File: 7segment.sch (KiCad schematic (older format))
At the start: 17 parts, among them J1 Conn_02x05_Counter_Clockwise

Commit message: Revision 3, reverse-mount regular 0805 UV LEDs
Parts:
- D1, D2, D3, D4, D5, D6, D7, D8: footprint LED_SMD:LED_0805_2012Metric -> LED_SMD:LED_0805_2012Metric_Pad1.15x1.40mm_HandSolder
Connections:
- net 9: now also R6.2; no longer D3.2 (A)
- net F: now also D3.2 (A), R6.1; no longer D3.1 (K), R6.2
- net GND: now also D3.1 (K); no longer R6.1
Changed lines of the file:
@@
 F 0 "D3" V 4039 3257 50  0000 R CNN
 F 1 "LED" V 3948 3257 50  0000 R CNN
-F 2 "LED_SMD:LED_0805_2012Metric" H 4000 3375 50  0001 C CNN
+F 2 "LED_SMD:LED_0805_2012Metric_Pad1.15x1.40mm_HandSolder" H 4000 3375 50  0001 C CNN
 F 3 "~" H 4000 3375 50  0001 C CNN
 	1    4000 3375
@@
 F 0 "D2" V 4789 3430 50  0000 L CNN
 F 1 "LED" V 4698 3430 50  0000 L CNN
-F 2 "LED_SMD:LED_0805_2012Metric" H 4750 3350 50  0001 C CNN
+F 2 "LED_SMD:LED_0805_2012Metric_Pad1.15x1.40mm_HandSolder" H 4750 3350 50  0001 C CNN
 F 3 "~" H 4750 3350 50  0001 C CNN
 	1    4750 3350
@@
 F 0 "D4" H 4368 3495 50  0000 C CNN
 F 1 "LED" H 4368 3586 50  0000 C CNN
-F 2 "LED_SMD:LED_0805_2012Metric" H 4375 3750 50  0001 C CNN
+F 2 "LED_SMD:LED_0805_2012Metric_Pad1.15x1.40mm_HandSolder" H 4375 3750 50  0001 C CNN
 F 3 "~" H 4375 3750 50  0001 C CNN
 	1    4375 3750
@@
 F 0 "D5" V 4039 4007 50  0000 R CNN
 F 1 "LED" V 3948 4007 50  0000 R CNN
-F 2 "LED_SMD:LED_0805_2012Metric" H 4000 4125 50  0001 C CNN
+F 2 "LED_SMD:LED_0805_2012Metric_Pad1.15x1.40mm_HandSolder" H 4000 4125 50  0001 C CNN
 F 3 "~" H 4000 4125 50  0001 C CNN
 	1    4000 4125
@@
 F 0 "D6" V 4789 4205 50  0000 L CNN
 F 1 "LED" V 4698 4205 50  0000 L CNN
-F 2 "LED_SMD:LED_0805_2012Metric" H 4750 4125 50  0001 C CNN
+F 2 "LED_SMD:LED_0805_2012Metric_Pad1.15x1.40mm_HandSolder" H 4750 4125 50  0001 C CNN
 F 3 "~" H 4750 4125 50  0001 C CNN
 	1    4750 4125
@@
 F 0 "D8" H 4368 4245 50  0000 C CNN
 F 1 "LED" H 4368 4336 50  0000 C CNN
-F 2 "LED_SMD:LED_0805_2012Metric" H 4375 4500 50  0001 C CNN
+F 2 "LED_SMD:LED_0805_2012Metric_Pad1.15x1.40mm_HandSolder" H 4375 4500 50  0001 C CNN
 F 3 "~" H 4375 4500 50  0001 C CNN
 	1    4375 4500
@@
 Text GLabel 4225 3000 0    50   Input ~ 0
 A
-Text GLabel 4000 3525 0    50   Input ~ 0
+Text GLabel 4000 3225 0    50   Input ~ 0
 F
 Text GLabel 4750 3200 0    50   Input ~ 0
@@
 F 0 "D7" V 5389 4430 50  0000 L CNN
 F 1 "LED" V 5298 4430 50  0000 L CNN
-F 2 "LED_SMD:LED_0805_2012Metric" H 5350 4350 50  0001 C CNN
+F 2 "LED_SMD:LED_0805_2012Metric_Pad1.15x1.40mm_HandSolder" H 5350 4350 50  0001 C CNN
 F 3 "~" H 5350 4350 50  0001 C CNN
 	1    5350 4350
@@
 Text GLabel 2425 3325 2    50   Input ~ 0
 E
-Text GLabel 2125 3500 0    50   Input ~ 0
+Text GLabel 2425 3500 2    50   Input ~ 0
 F
 Text GLabel 2425 3675 2    50   Input ~ 0
@@
 Text GLabel 2125 3325 0    50   Input ~ 0
 1
-Text GLabel 4000 3225 0    50   Input ~ 0
+Text GLabel 2125 3500 0    50   Input ~ 0
 9
 Text GLabel 2125 3675 0    50   Input ~ 0
@@
 Text GLabel 4525 3750 2    50   Input ~ 0
 GND
-Text GLabel 2425 3500 2    50   Input ~ 0
+Text GLabel 4000 3525 0    50   Input ~ 0
 GND
 Text GLabel 4000 4275 0    50   Input ~ 0
@@
 F 0 "D1" H 4368 2745 50  0000 C CNN
 F 1 "LED" H 4368 2836 50  0000 C CNN
-F 2 "LED_SMD:LED_0805_2012Metric" H 4375 3000 50  0001 C CNN
+F 2 "LED_SMD:LED_0805_2012Metric_Pad1.15x1.40mm_HandSolder" H 4375 3000 50  0001 C CNN
 F 3 "~" H 4375 3000 50  0001 C CNN
 	1    4375 3000
